File: schematic/blinkm_mk2j.brd (EAGLE design)
At the start: 15.8 x 17.8 mm, 16 parts, among them CN1 1X4SMT, Q1 MOSFET-PCHANNELIRLML2244, SW1 SPST_TACT-KMR2, SW2 SPST_TACT-KMR2, U1 ATTINY44QFN

Commit message: more better
Parts:
- moved LED1 9.40 mm to (12.4, 13.2)
- moved LED2 8.39 mm to (7.87, 6.60), turned to 180 degrees
- moved LED3 7.98 mm to (3.05, 13.2), turned to 90 degrees
- moved C1 0.51 mm to (6.35, 4.83)
- moved C2 0.51 mm to (8.38, 4.83)
- moved R1 0.51 mm to (4.57, 4.83)
Connections:
- net N$1 renamed DOI1
- net N$2 renamed DOI2
- net DO: now also CN1.3; no longer CN1.2
- net VCC: now also CN1.2; no longer CN1.3
Routing:
- net DI: track 19.5 -> 4.94 mm
- net RESET: track 15.7 -> 27.9 mm, vias 2 -> 3
- net DOI1: track 9.96 -> 18.7 mm
- net DO: track 15.0 -> 6.66 mm
- net LEDEN: track 4.92 -> 12.4 mm
- net SDA: track 21.7 -> 16.6 mm, vias 2 -> 1
- net GND: track 71.6 -> 68.0 mm, vias 8 -> 7
- net SCL: track 9.40 -> 12.5 mm, vias 1 -> 2
- net +5V: track 45.9 -> 43.1 mm, vias 1 -> 3
- net A1: track 13.7 -> 16.3 mm, vias 1 -> 2
- net A0: track 11.1 -> 12.6 mm, vias 1 -> 2
- net DOI2: track 5.40 -> 6.71 mm
- net MISO: track 12.7 -> 11.5 mm, vias 1 -> 2
- net VCC: track 19.1 -> 18.5 mm, vias 3 -> 1
Other:
- board text added: "do"
- board text added: "gnd"
- board text removed: "Gnd"
