File: schematic/blinkm_mk2j.sch (EAGLE design)
At the start: 18 parts, among them CN1 1X4SMT, U1 ATTINY44QFN

Commit message: sync
Parts:
- removed C5, C6: 100nF, rcl:C-USC0603
- removed LED4: WS2812B, WS2812:WS2812B
- removed TP1, TP2: TEST-POINT3, SparkFun-Passives:TEST-POINT3
- added Q1: MOSFET-PCHANNELIRLML2244, SparkFun-DiscreteSemi:MOSFET-PCHANNELIRLML2244
- added SW1, SW2: SPST_TACT-KMR2, adafruit:SPST_TACT-KMR2
Connections:
- removed net N$12: U1.PB0
- removed net N$13: U1.PB1
- removed net N$14: U1.PB2
- removed net N$3: LED3.DO, LED4.DI
- removed net N$6: U1.PA2/ADC2
- removed net N$7: U1.PA3/ADC3
- new net LEDEN: Q1.G, U1.PA3/ADC3
- new net VCC: CN1.3, LED1.VDD, LED2.VDD, LED3.VDD, Q1.S
- net +5V: now also Q1.D; no longer C5.1, C6.1, CN1.3, LED1.VDD, LED2.VDD, LED3.VDD, LED4.VDD
- net A0: now also SW1.P, SW1.P1
- net A1: now also SW2.P, SW2.P1
- net DI: no longer TP1.1
- net DO: now also LED3.DO; no longer LED4.DO
- net GND: now also SW1.S, SW1.S1, SW2.S, SW2.S1; no longer C5.2, C6.2, LED4.VSS, TP2.1
Other:
- note removed: "SWITCH-MOMENTARY-2SMD-2"

Commit message: more better
Connections:
- net N$1 renamed DOI1
- net N$2 renamed DOI2
- net DO: now also CN1.3; no longer CN1.2
- net VCC: now also CN1.2; no longer CN1.3
Changed lines of the file:
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@@
 <instance part="SUPPLY2" gate="1" x="220.98" y="154.94"/>
 <instance part="SUPPLY3" gate="1" x="220.98" y="134.62"/>
-<instance part="SUPPLY4" gate="1" x="149.86" y="172.72"/>
+<instance part="SUPPLY4" gate="1" x="152.4" y="175.26"/>
 <instance part="SW1" gate="G$1" x="96.52" y="50.8" rot="R270"/>
 <instance part="GND18" gate="1" x="101.6" y="43.18"/>
@@
 </segment>
 <segment>
-<pinref part="CN1" gate="G$1" pin="2"/>
-<wire x1="160.02" y1="172.72" x2="154.94" y2="172.72" width="0.1524" layer="91"/>
-<label x="154.94" y="172.72" size="1.778" layer="95"/>
+<pinref part="CN1" gate="G$1" pin="3"/>
+<wire x1="160.02" y1="170.18" x2="152.4" y2="170.18" width="0.1524" layer="91"/>
+<label x="152.4" y="170.18" size="1.778" layer="95"/>
 </segment>
 </net>
@@
 </segment>
 </net>
-<net name="N$1" class="0">
+<net name="DOI1" class="0">
 <segment>
 <pinref part="LED1" gate="G$1" pin="DO"/>
@@
 </segment>
 <segment>
-<pinref part="CN1" gate="G$1" pin="3"/>
-<wire x1="160.02" y1="170.18" x2="149.86" y2="170.18" width="0.1524" layer="91"/>
-<wire x1="149.86" y1="170.18" x2="149.86" y2="172.72" width="0.1524" layer="91"/>
-<pinref part="SUPPLY4" gate="1" pin="VCC"/>
-</segment>
-<segment>
 <pinref part="LED3" gate="G$1" pin="VDD"/>
 <pinref part="SUPPLY5" gate="1" pin="VCC"/>
 <wire x1="220.98" y1="114.3" x2="223.52" y2="114.3" width="0.1524" layer="91"/>
 </segment>
+<segment>
+<pinref part="CN1" gate="G$1" pin="2"/>
+<pinref part="SUPPLY4" gate="1" pin="VCC"/>
+<wire x1="160.02" y1="172.72" x2="152.4" y2="172.72" width="0.1524" layer="91"/>
+<wire x1="152.4" y1="172.72" x2="152.4" y2="175.26" width="0.1524" layer="91"/>
+</segment>
 </net>
 <net name="LEDEN" class="0">
@@
 </segment>
 </net>
-<net name="N$2" class="0">
+<net name="DOI2" class="0">
 <segment>
 <pinref part="LED2" gate="G$1" pin="DO"/>
