File: schematic/blinkm_mk2r.brd (EAGLE design)
At the start: 17.8 x 19.1 mm, 15 parts, among them CN1 1X4SMT, CN2 1X4SMT, CN3 1X4SMT, Q1 MOSFET-PCHANNELIRLML2244, U1 ATTINY44QFN

Commit message: woot, hopefully figured out smaller algo for fading
Parts:
- turned Q1 to 0 degrees
Connections:
- net +5V: now also Q1.2; no longer Q1.3
- net VCC: now also Q1.3; no longer Q1.2
Routing:
- net +5V: track 50.0 -> 48.1 mm
- net LEDEN: track 14.3 -> 15.8 mm
- net N$2: track 5.49 -> 6.81 mm
- net GND: track 68.4 -> 67.1 mm
- net VCC: track 30.0 -> 31.1 mm
- net SDA: track 6.83 -> 7.34 mm
