File: schematic/blinkm_mk2r.sch (EAGLE design)
At the start: 15 parts, among them CN1 1X4SMT, CN2 1X4SMT, CN3 1X4SMT, Q1 MOSFET-PCHANNELIRLML2244, U1 ATTINY44QFN

Commit message: woot, hopefully figured out smaller algo for fading
Connections:
- net +5V: now also Q1.S; no longer Q1.D
- net VCC: now also Q1.D; no longer Q1.S
Other:
- moved on the sheet: Q1
Changed lines of the file:
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@@
 <attribute name="VALUE" x="33.02" y="106.68" size="1.778" layer="96" rot="R180"/>
 </instance>
-<instance part="Q1" gate="G$1" x="154.94" y="134.62"/>
-<instance part="P+7" gate="1" x="154.94" y="144.78" smashed="yes">
-<attribute name="VALUE" x="157.48" y="147.32" size="1.778" layer="96" rot="R180"/>
+<instance part="Q1" gate="G$1" x="162.56" y="129.54" rot="R270"/>
+<instance part="P+7" gate="1" x="144.78" y="132.08" smashed="yes">
+<attribute name="VALUE" x="147.32" y="134.62" size="1.778" layer="96" rot="R180"/>
 </instance>
-<instance part="SUPPLY1" gate="1" x="165.1" y="127"/>
+<instance part="SUPPLY1" gate="1" x="180.34" y="129.54"/>
 <instance part="SUPPLY2" gate="1" x="220.98" y="154.94"/>
 <instance part="SUPPLY3" gate="1" x="220.98" y="134.62"/>
@@
 </segment>
 <segment>
-<pinref part="Q1" gate="G$1" pin="D"/>
-<pinref part="P+7" gate="1" pin="+5V"/>
-<wire x1="154.94" y1="139.7" x2="154.94" y2="142.24" width="0.1524" layer="91"/>
-</segment>
-<segment>
 <pinref part="CN2" gate="G$1" pin="1"/>
 <pinref part="P+10" gate="1" pin="+5V"/>
@@
 <pinref part="P+9" gate="1" pin="+5V"/>
 <wire x1="116.84" y1="172.72" x2="111.76" y2="172.72" width="0.1524" layer="91"/>
+</segment>
+<segment>
+<pinref part="P+7" gate="1" pin="+5V"/>
+<pinref part="Q1" gate="G$1" pin="S"/>
+<wire x1="144.78" y1="129.54" x2="157.48" y2="129.54" width="0.1524" layer="91"/>
 </segment>
 </net>
@@
 <net name="VCC" class="0">
 <segment>
-<pinref part="SUPPLY1" gate="1" pin="VCC"/>
-<wire x1="165.1" y1="127" x2="165.1" y2="124.46" width="0.1524" layer="91"/>
-<pinref part="Q1" gate="G$1" pin="S"/>
-<wire x1="154.94" y1="129.54" x2="154.94" y2="124.46" width="0.1524" layer="91"/>
-<wire x1="154.94" y1="124.46" x2="160.02" y2="124.46" width="0.1524" layer="91"/>
-<label x="157.48" y="124.46" size="1.778" layer="95"/>
-<wire x1="165.1" y1="124.46" x2="160.02" y2="124.46" width="0.1524" layer="91"/>
-</segment>
-<segment>
 <wire x1="223.52" y1="154.94" x2="220.98" y2="154.94" width="0.1524" layer="91"/>
 <pinref part="LED1" gate="G$1" pin="VDD"/>
@@
 <wire x1="220.98" y1="93.98" x2="223.52" y2="93.98" width="0.1524" layer="91"/>
 </segment>
+<segment>
+<pinref part="Q1" gate="G$1" pin="D"/>
+<pinref part="SUPPLY1" gate="1" pin="VCC"/>
+<wire x1="167.64" y1="129.54" x2="180.34" y2="129.54" width="0.1524" layer="91"/>
+</segment>
 </net>
 <net name="LEDEN" class="0">
 <segment>
 <pinref part="Q1" gate="G$1" pin="G"/>
-<wire x1="147.32" y1="134.62" x2="137.16" y2="134.62" width="0.1524" layer="91"/>
-<label x="137.16" y="134.62" size="1.778" layer="95"/>
-</segment>
-<segment>
+<wire x1="162.56" y1="137.16" x2="162.56" y2="142.24" width="0.1524" layer="91"/>
+<label x="152.4" y="142.24" size="1.778" layer="95"/>
+<wire x1="162.56" y1="142.24" x2="152.4" y2="142.24" width="0.1524" layer="91"/>
+</segment>
+<segment>
