File: schematic/blinkm_mk2s.sch (EAGLE design)
At the start: 9 parts, among them CN1 1X4SMT, Q1 MOSFET-PCHANNELIRLML2244, U1 ATTINY44QFN

Commit message: update before sketching15
Parts:
- Q1: value MOSFET-PCHANNELIRLML2244 -> MOSFET-PCHAN
Other:
- note added: "LED"
- note added: "RAW"
- note added: "VCC"
Changed lines of the file:
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@@
 <part name="GND2" library="SparkFun-20110517" deviceset="GND" device=""/>
 <part name="P+5" library="supply1" deviceset="+5V" device=""/>
-<part name="Q1" library="SparkFun-DiscreteSemi" deviceset="MOSFET-PCHANNEL" device="IRLML2244"/>
+<part name="Q1" library="SparkFun-DiscreteSemi" deviceset="MOSFET-PCHANNEL" device="IRLML2244" value="MOSFET-PCHAN"/>
 <part name="P+7" library="supply1" deviceset="+5V" device=""/>
 <part name="SUPPLY1" library="SparkFun-Aesthetics" deviceset="VCC" device=""/>
@@
 <sheet>
 <plain>
+<text x="171.704" y="115.316" size="1.778" layer="95">LED</text>
+<text x="135.382" y="113.03" size="1.778" layer="95">VCC</text>
+<text x="135.382" y="115.57" size="1.778" layer="95">RAW</text>
 </plain>
 <instances>
@@
 <attribute name="VALUE" x="66.04" y="104.14" size="1.778" layer="96" rot="R180"/>
 </instance>
-<instance part="Q1" gate="G$1" x="162.56" y="99.06" rot="R270"/>
-<instance part="P+7" gate="1" x="137.16" y="101.6" smashed="yes">
-<attribute name="VALUE" x="139.7" y="104.14" size="1.778" layer="96" rot="R180"/>
+<instance part="Q1" gate="G$1" x="162.56" y="99.06" smashed="yes" rot="R270">
+<attribute name="NAME" x="156.972" y="95.504" size="1.778" layer="95"/>
+<attribute name="VALUE" x="156.718" y="92.456" size="1.778" layer="96"/>
+</instance>
+<instance part="P+7" gate="1" x="137.16" y="111.76" smashed="yes">
+<attribute name="VALUE" x="134.62" y="124.46" size="1.778" layer="96"/>
 </instance>
 <instance part="SUPPLY1" gate="1" x="172.72" y="109.22"/>
@@
 <pinref part="Q1" gate="G$1" pin="S"/>
 <pinref part="P+7" gate="1" pin="+5V"/>
+<wire x1="137.16" y1="109.22" x2="137.16" y2="99.06" width="0.1524" layer="91"/>
 <wire x1="137.16" y1="99.06" x2="157.48" y2="99.06" width="0.1524" layer="91"/>
 </segment>
@@
 <segment>
 <pinref part="Q1" gate="G$1" pin="G"/>
-<wire x1="162.56" y1="106.68" x2="144.78" y2="106.68" width="0.1524" layer="91"/>
-<label x="147.32" y="106.68" size="1.778" layer="95"/>
-</segment>
-<segment>
+<wire x1="162.56" y1="106.68" x2="162.56" y2="109.22" width="0.1524" layer="91"/>
+<wire x1="162.56" y1="109.22" x2="149.86" y2="109.22" width="0.1524" layer="91"/>
+<label x="152.4" y="109.22" size="1.778" layer="95"/>
+</segment>
+<segment>
