File: schematic/blinkm2neo_5Jul2020_qfn.brd (EAGLE design)
At the start: 13.2 x 13.3 mm, 10 parts, among them IC1 ATTINY85SOIC, J1 blinkm

Commit message: added pullup resistors
Parts:
- added JP1: JUMPER-SMT_2_NC_TRACE_NO-SILK, SparkFun-Jumpers:SMT-JUMPER_2_NC_TRACE_NO-SILK
- added R2, R3: 10k, SparkFun-Resistors:0402
- J2: value (none) -> neopixel
- J3: value (none) -> reset
- J4: value (none) -> miso
- R1: value (none) -> 200
Connections:
- new net N$1: JP1.2, R2.1, R3.1
- net SCL: now also R2.2
- net SDA: now also R3.2
- net VCC: now also JP1.1
Routing:
- net SCL: track 6.58 -> 14.0 mm
- net SDA: track 4.73 -> 7.79 mm
- net N$1: track 0.00 -> 2.84 mm
- net VCC: track 4.71 -> 6.19 mm, vias 0 -> 1
- net GND: track 13.0 -> 14.2 mm
Other:
- board text added: "pull"
